File: biym-board/motor.kicad_sch (KiCad schematic)
At the start: 0 parts

Commit message: More motor driver wiring
Parts:
- added U?: DRV8311H, Janelia:WQFN-24-1EP_3x3mm_P0.4mm_EP1.9x1.9mm_ThermalVias, symbol Janelia:DRV8311H
Connections:
- new net GND: U?.16 (AGND), U?.25 (PAD), U?.9 (PGND)
- new net MOTOR_A: U?.10 (OUTA)
- new net MOTOR_B: U?.11 (OUTB)
- new net MOTOR_C: U?.12 (OUTC)
- new net PWM_A: U?.15 (INHA)
- new net PWM_B: U?.14 (INHB)
- new net PWM_C: U?.13 (INHC)
- new net VDIGITAL: U?.18 (INLA), U?.19 (INLB), U?.20 (INLC), U?.7 (VIN_AVDD)
- new net VMOTOR: U?.8 (VM)
- new net ~{SLEEP}: U?.24 (~{SLEEP})
- no-connect marks 0 -> 6
Other:
- note added: "Gain: 1 V/A"
- note added: "Mode: 3x PWM and 9A OCP Level"
- note added: "Slew: 180 V/us"
Changed lines of the file:
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@@
     (rev "0.1")
   )
+  (junction (at 116.84 85.09) (diameter 0) (color 0 0 0 0)
+  )
+  (junction (at 134.62 113.03) (diameter 0) (color 0 0 0 0)
+  )
+  (no_connect (at 119.38 102.87))
+  (no_connect (at 149.86 87.63))
+  (no_connect (at 149.86 90.17))
+  (no_connect (at 119.38 97.79))
+  (no_connect (at 149.86 92.71))
+  (no_connect (at 119.38 100.33))
+  (wire (pts (xy 137.16 110.49) (xy 137.16 113.03))
+    (stroke (width 0) (type default) (color 0 0 0 0))
+  )
+  (wire (pts (xy 149.86 80.01) (xy 152.4 80.01))
+    (stroke (width 0) (type default) (color 0 0 0 0))
+  )
+  (wire (pts (xy 64.77 82.55) (xy 67.31 82.55))
+    (stroke (width 0) (type default) (color 0 0 0 0))
+  )
+  (wire (pts (xy 116.84 87.63) (xy 119.38 87.63))
+    (stroke (width 0) (type default) (color 0 0 0 0))
+  )
+  (wire (pts (xy 116.84 82.55) (xy 116.84 85.09))
+    (stroke (width 0) (type default) (color 0 0 0 0))
+  )
+  (wire (pts (xy 138.43 52.07) (xy 138.43 54.61))
+    (stroke (width 0) (type default) (color 0 0 0 0))
+  )
+  (wire (pts (xy 132.08 113.03) (xy 134.62 113.03))
+    (stroke (width 0) (type default) (color 0 0 0 0))
+  )
+  (wire (pts (xy 149.86 74.93) (xy 152.4 74.93))
+    (stroke (width 0) (type default) (color 0 0 0 0))
+  )
+  (wire (pts (xy 119.38 82.55) (xy 116.84 82.55))
+    (stroke (width 0) (type default) (color 0 0 0 0))
+  )
+  (wire (pts (xy 116.84 85.09) (xy 119.38 85.09))
+    (stroke (width 0) (type default) (color 0 0 0 0))
+  )
+  (wire (pts (xy 134.62 113.03) (xy 134.62 115.57))
+    (stroke (width 0) (type default) (color 0 0 0 0))
+  )
+  (wire (pts (xy 116.84 85.09) (xy 116.84 87.63))
+    (stroke (width 0) (type default) (color 0 0 0 0))
+  )
+  (wire (pts (xy 116.84 74.93) (xy 119.38 74.93))
+    (stroke (width 0) (type default) (color 0 0 0 0))
+  )
+  (wire (pts (xy 116.84 72.39) (xy 119.38 72.39))
+    (stroke (width 0) (type default) (color 0 0 0 0))
+  )
+  (wire (pts (xy 114.3 85.09) (xy 116.84 85.09))
+    (stroke (width 0) (type default) (color 0 0 0 0))
+  )
+  (wire (pts (xy 116.84 77.47) (xy 119.38 77.47))
+    (stroke (width 0) (type default) (color 0 0 0 0))
+  )
+  (wire (pts (xy 116.84 92.71) (xy 119.38 92.71))
+    (stroke (width 0) (type default) (color 0 0 0 0))
+  )
+  (wire (pts (xy 132.08 110.49) (xy 132.08 113.03))
+    (stroke (width 0) (type default) (color 0 0 0 0))
+  )
+  (wire (pts (xy 149.86 77.47) (xy 152.4 77.47))
+    (stroke (width 0) (type default) (color 0 0 0 0))
+  )
+  (wire (pts (xy 64.77 85.09) (xy 67.31 85.09))
+    (stroke (width 0) (type default) (color 0 0 0 0))
+  )
+  (wire (pts (xy 64.77 87.63) (xy 67.31 87.63))
+    (stroke (width 0) (type default) (color 0 0 0 0))
+  )
+  (wire (pts (xy 134.62 110.49) (xy 134.62 113.03))
+    (stroke (width 0) (type default) (color 0 0 0 0))
+  )
+  (wire (pts (xy 134.62 113.03) (xy 137.16 113.03))
+    (stroke (width 0) (type default) (color 0 0 0 0))
+  )
+  (wire (pts (xy 130.81 52.07) (xy 130.81 54.61))
+    (stroke (width 0) (type default) (color 0 0 0 0))
+  )
+  (text "Gain: 1 V/A" (at 114.3 102.87 180)
+    (effects (font (size 1.27 1.27)) (justify right bottom))
+  )
+  (text "Slew: 180 V/us" (at 114.3 100.33 180)
+    (effects (font (size 1.27 1.27)) (justify right bottom))
+  )
+  (text "Mode: 3x PWM and 9A OCP Level" (at 114.3 97.79 180)
+    (effects (font (size 1.27 1.27)) (justify right bottom))
+  )
+  (label "VMOTOR" (at 67.31 82.55 0)
+    (effects (font (size 1.27 1.27)) (justify left bottom))
+  )
+  (label "VMOTOR" (at 138.43 52.07 0)
+    (effects (font (size 1.27 1.27)) (justify left bottom))
+  )
+  (label "GND" (at 134.62 115.57 0)
+    (effects (font (size 1.27 1.27)) (justify left bottom))
+  )
+  (label "MOTOR_B" (at 152.4 77.47 0)
+    (effects (font (size 1.27 1.27)) (justify left bottom))
+  )
+  (label "GND" (at 67.31 87.63 0)
+    (effects (font (size 1.27 1.27)) (justify left bottom))
+  )
+  (label "VDIGITAL" (at 130.81 52.07 180)
+    (effects (font (size 1.27 1.27)) (justify right bottom))
+  )
+  (label "MOTOR_A" (at 152.4 74.93 0)
+    (effects (font (size 1.27 1.27)) (justify left bottom))
+  )
+  (label "MOTOR_C" (at 152.4 80.01 0)
+    (effects (font (size 1.27 1.27)) (justify left bottom))
+  )
+  (label "VDIGITAL" (at 114.3 85.09 180)
+    (effects (font (size 1.27 1.27)) (justify right bottom))
+  )
+  (label "VDIGITAL" (at 67.31 85.09 0)
+    (effects (font (size 1.27 1.27)) (justify left bottom))
+  )
+  (hierarchical_label "PWM_A" (shape input) (at 116.84 72.39 180)
+    (effects (font (size 1.27 1.27)) (justify right))
+  )
+  (hierarchical_label "VDIGITAL" (shape passive) (at 64.77 85.09 180)
+    (effects (font (size 1.27 1.27)) (justify right))
+  )
+  (hierarchical_label "~{SLEEP}" (shape input) (at 116.84 92.71 180)
+    (effects (font (size 1.27 1.27)) (justify right))
+  )
+  (hierarchical_label "GND" (shape passive) (at 64.77 87.63 180)
+    (effects (font (size 1.27 1.27)) (justify right))
+  )
+  (hierarchical_label "VMOTOR" (shape passive) (at 64.77 82.55 180)
+    (effects (font (size 1.27 1.27)) (justify right))
+  )
+  (hierarchical_label "PWM_C" (shape input) (at 116.84 77.47 180)
+    (effects (font (size 1.27 1.27)) (justify right))
+  )
+  (hierarchical_label "PWM_B" (shape input) (at 116.84 74.93 180)
+    (effects (font (size 1.27 1.27)) (justify right))
+  )
+  (symbol (lib_id "Janelia:DRV8311H") (at 134.62 82.55 0) (unit 1)
+    (in_bom yes) (on_board yes)
+    (property "Reference" "U?" (id 0) (at 142.24 58.42 0)
+      (effects (font (size 1.524 1.524)) (justify left))
+    )
+    (property "Value" "DRV8311H" (id 1) (at 137.16 106.68 0)
+      (effects (font (size 1.524 1.524)) (justify left))
+    )
+    (property "Footprint" "Janelia:WQFN-24-1EP_3x3mm_P0.4mm_EP1.9x1.9mm_ThermalVias" (id 2) (at 134.62 27.94 0)
+      (effects (font (size 1.524 1.524)) hide)
+    )
+    (property "Datasheet" "" (id 3) (at 193.04 44.45 0)
+      (effects (font (size 1.524 1.524)) hide)
+    )
+    (property "Vendor Part Number" "296-DRV8311HRRWRCT-ND" (id 4) (at 134.62 35.56 0)
+      (effects (font (size 1.524 1.524)) hide)
+    )
+    (property "Description" "24V ABS MAX 3 TO 20V 3-PHASE B" (id 5) (at 134.62 33.02 0)
+      (effects (font (size 1.524 1.524)) hide)
+    )
+    (property "Vendor" "Digi-Key" (id 6) (at 134.62 30.48 0)
+      (effects (font (size 1.524 1.524)) hide)
+    )
+    (property "Manufacturer" "Texas Instruments" (id 7) (at 134.62 38.1 0)
+      (effects (font (size 1.27 1.27)) hide)
+    )
+    (property "Manufacturer Part Number" "DRV8311HRRWR" (id 8) (at 134.62 25.4 0)
+      (effects (font (size 1.27 1.27)) hide)
+    )
+    (pin "1")
+    (pin "10")
+    (pin "11")
+    (pin "12")
+    (pin "13")
+    (pin "14")
+    (pin "15")
+    (pin "16")
+    (pin "17")
+    (pin "18")
+    (pin "19")
+    (pin "2")
+    (pin "20")
+    (pin "21")
+    (pin "22")
+    (pin "23")
+    (pin "24")
+    (pin "25")
+    (pin "3")
+    (pin "4")
+    (pin "5")
+    (pin "6")
+    (pin "7")
+    (pin "8")
+    (pin "9")
+  )
 )
