File: biym-board/motor_driver.kicad_sch (KiCad schematic)
At the start: 1 part

Commit message: Rename reference files
Parts:
- added J?: HEADER_01X03_JST_PH_VERTICAL, Janelia:JST_PH_B3B-PH-K_1x03_P2.00mm_Vertical, symbol Janelia:HEADER_01X03_JST_PH_VERTICAL
Connections:
- net MOTOR_A: now also J?.1 (Pin_1)
- net MOTOR_B: now also J?.2 (Pin_2)
- net MOTOR_C: now also J?.3 (Pin_3)
- net ~{FAULT}: now reaches U?.1 (~{FAULT})
- net VDD: now reaches U?.17 (AVDD)
- net CSAREF: now reaches U?.2 (CSAREF)
- net CP: now reaches U?.6 (CP)
- net VMOTOR renamed VDRIVER
Changed lines of the file:
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@@
+    (stroke (width 0) (type default) (color 0 0 0 0))
+  )
+  (wire (pts (xy 149.86 64.77) (xy 152.4 64.77))
+    (stroke (width 0) (type default) (color 0 0 0 0))
+  )
+  (wire (pts (xy 149.86 97.79) (xy 152.4 97.79))
     (stroke (width 0) (type default) (color 0 0 0 0))
   )
@@
     (stroke (width 0) (type default) (color 0 0 0 0))
   )
+  (wire (pts (xy 204.47 80.01) (xy 207.01 80.01))
+    (stroke (width 0) (type default) (color 0 0 0 0))
+  )
+  (wire (pts (xy 149.86 83.82) (xy 152.4 83.82))
+    (stroke (width 0) (type default) (color 0 0 0 0))
+  )
+  (wire (pts (xy 149.86 69.85) (xy 152.4 69.85))
+    (stroke (width 0) (type default) (color 0 0 0 0))
+  )
   (wire (pts (xy 134.62 113.03) (xy 134.62 115.57))
     (stroke (width 0) (type default) (color 0 0 0 0))
@@
   )
   (wire (pts (xy 116.84 74.93) (xy 119.38 74.93))
+    (stroke (width 0) (type default) (color 0 0 0 0))
+  )
+  (wire (pts (xy 204.47 77.47) (xy 207.01 77.47))
     (stroke (width 0) (type default) (color 0 0 0 0))
   )
@@
     (stroke (width 0) (type default) (color 0 0 0 0))
   )
+  (wire (pts (xy 204.47 74.93) (xy 207.01 74.93))
+    (stroke (width 0) (type default) (color 0 0 0 0))
+  )
   (wire (pts (xy 134.62 110.49) (xy 134.62 113.03))
     (stroke (width 0) (type default) (color 0 0 0 0))
@@
     (effects (font (size 1.27 1.27)) (justify right bottom))
   )
-  (label "VMOTOR" (at 67.31 82.55 0)
+  (label "VDRIVER" (at 67.31 82.55 0)
     (effects (font (size 1.27 1.27)) (justify left bottom))
   )
-  (label "VMOTOR" (at 138.43 52.07 0)
+  (label "CSAREF" (at 152.4 97.79 0)
+    (effects (font (size 1.27 1.27)) (justify left bottom))
+  )
+  (label "CP" (at 152.4 64.77 0)
+    (effects (font (size 1.27 1.27)) (justify left bottom))
+  )
+  (label "VDRIVER" (at 138.43 52.07 0)
     (effects (font (size 1.27 1.27)) (justify left bottom))
   )
@@
     (effects (font (size 1.27 1.27)) (justify left bottom))
   )
+  (label "VDD" (at 152.4 69.85 0)
+    (effects (font (size 1.27 1.27)) (justify left bottom))
+  )
   (label "MOTOR_B" (at 152.4 77.47 0)
     (effects (font (size 1.27 1.27)) (justify left bottom))
   )
+  (label "MOTOR_C" (at 207.01 80.01 0)
+    (effects (font (size 1.27 1.27)) (justify left bottom))
+  )
+  (label "MOTOR_A" (at 207.01 74.93 0)
+    (effects (font (size 1.27 1.27)) (justify left bottom))
+  )
+  (label "~{FAULT}" (at 152.4 83.82 0)
+    (effects (font (size 1.27 1.27)) (justify left bottom))
+  )
   (label "GND" (at 67.31 87.63 0)
+    (effects (font (size 1.27 1.27)) (justify left bottom))
+  )
+  (label "MOTOR_B" (at 207.01 77.47 0)
     (effects (font (size 1.27 1.27)) (justify left bottom))
   )
@@
     (effects (font (size 1.27 1.27)) (justify right))
   )
-  (hierarchical_label "VMOTOR" (shape passive) (at 64.77 82.55 180)
+  (hierarchical_label "VDRIVER" (shape passive) (at 64.77 82.55 180)
     (effects (font (size 1.27 1.27)) (justify right))
   )
@@
     (effects (font (size 1.27 1.27)) (justify right))
   )
+  (symbol (lib_id "Janelia:HEADER_01X03_JST_PH_VERTICAL") (at 199.39 77.47 0) (unit 1)
+    (in_bom yes) (on_board yes)
+    (property "Reference" "J?" (id 0) (at 199.39 72.39 0))
+    (property "Value" "HEADER_01X03_JST_PH_VERTICAL" (id 1) (at 199.39 82.55 0))
+    (property "Footprint" "Janelia:JST_PH_B3B-PH-K_1x03_P2.00mm_Vertical" (id 2) (at 199.39 64.77 0)
+      (effects (font (size 1.27 1.27)) hide)
+    )
+    (property "Datasheet" "" (id 3) (at 199.39 77.47 0)
+      (effects (font (size 1.27 1.27)) hide)
+    )
+    (property "Description" "CONN HEADER VERT 3POS 2MM" (id 4) (at 199.39 67.31 0)
+      (effects (font (size 1.27 1.27)) hide)
+    )
+    (property "Manufacturer" "JST Sales America Inc." (id 5) (at 199.39 59.69 0)
+      (effects (font (size 1.27 1.27)) hide)
+    )
+    (property "Manufacturer Part Number" "B3B-PH-K-S(LF)(SN)" (id 6) (at 199.39 62.23 0)
+      (effects (font (size 1.27 1.27)) hide)
+    )
+    (property "Vendor" "Digi-Key" (id 7) (at 199.39 57.15 0)
+      (effects (font (size 1.27 1.27)) hide)
+    )
+    (property "Vendor Part Number" "455-1705-ND" (id 8) (at 199.39 54.61 0)
+      (effects (font (size 1.27 1.27)) hide)
+    )
+    (pin "1")
+    (pin "2")
+    (pin "3")
+  )
   (symbol (lib_id "Janelia:DRV8311H") (at 134.62 82.55 0) (unit 1)

Commit message: Add driver external components
Parts:
- added C1, C3, C4, C7: 0.1uF, Janelia:SM0402, symbol Janelia:0.1uF_0402
- added C2, C5: 10uF, Janelia:SM0402_POL, symbol Janelia:10uF_0402_POL
- added C6: 1uF, Janelia:SM0402_POL, symbol Janelia:1uF_0402_POL
- added R2: 5.1k, Janelia:SM0402, symbol Janelia:5.1k_0402
- gave numbers to parts that had none: 2
Connections:
- net CP: now also C3.2
- net CSAREF: now also C7.1
- net GND: now also C1.2, C2.2, C4.2, C5.2, C6.2, C7.2
- net VDD: now also C6.1
- net VDIGITAL: now also C4.1, C5.1, R2.1
- net VDRIVER: now also C1.1, C2.1, C3.1
- net ~{FAULT}: now also R2.2
Other:
- moved on the sheet: J2, U1
