File: biym-board/encoder.kicad_sch (KiCad schematic)
At the start: 2 parts, among them U2 AS5047P

Commit message: Rename sheets
Connections:
- net ENCODER_A renamed A
- net ENCODER_B renamed B
Changed lines of the file:
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@@
     (effects (font (size 1.27 1.27)) (justify right))
   )
-  (hierarchical_label "ENCODER_B" (shape output) (at 147.32 90.17 0)
+  (hierarchical_label "B" (shape output) (at 147.32 90.17 0)
     (effects (font (size 1.27 1.27)) (justify left))
   )
@@
     (effects (font (size 1.27 1.27)) (justify right))
   )
-  (hierarchical_label "ENCODER_A" (shape output) (at 147.32 87.63 0)
+  (hierarchical_label "A" (shape output) (at 147.32 87.63 0)
     (effects (font (size 1.27 1.27)) (justify left))
   )

Commit message: Wire led sheet
Connections:
- net MISO: now also U2.3 (MISO); no longer U2.4 (MOSI)
- net MOSI: now also U2.4 (MOSI); no longer U2.3 (MISO)
Changed lines of the file:
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@@
     (effects (font (size 1.27 1.27)) (justify right))
   )
-  (hierarchical_label "MOSI" (shape output) (at 111.76 95.25 180)
+  (hierarchical_label "MISO" (shape output) (at 111.76 95.25 180)
     (effects (font (size 1.27 1.27)) (justify right))
   )
@@
     (effects (font (size 1.27 1.27)) (justify left))
   )
-  (hierarchical_label "MISO" (shape input) (at 111.76 92.71 180)
+  (hierarchical_label "MOSI" (shape input) (at 111.76 92.71 180)
     (effects (font (size 1.27 1.27)) (justify right))
   )

Commit message: Finished v0.1 of schematic
Parts:
- removed C8: 0.1uF, Janelia:SM0402, symbol Janelia:0.1uF_0402
- added C11: C_0.1uF_0402, Janelia:SM0402, symbol Janelia:C_0.1uF_0402
- renumbered U2 to U3
Connections:
- net GND: now also C11.2
- net VDIGITAL: now also C11.1
Other:
- company: (none) -> Peter Polidoro
- title: (none) -> biym-board-encoder
Changed lines of the file:
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@@
 (kicad_sch (version 20211123) (generator eeschema)
   (paper "A4")
+  (title_block
+    (title "biym-board-encoder")
+    (date "2022-11-17")
+    (rev "0.1")
+    (company "Peter Polidoro")
+  )
   (junction (at 129.54 118.11) (diameter 0) (color 0 0 0 0)
   )
@@
     (effects (font (size 1.27 1.27)) (justify right))
   )
+  (symbol (lib_id "Janelia:C_0.1uF_0402") (at 152.4 60.96 0) (unit 1)
+    (in_bom yes) (on_board yes)
+    (property "Reference" "C11" (id 0) (at 154.94 58.42 0)
+      (effects (font (size 1.016 1.016)) (justify left))
+    )
+    (property "Value" "C_0.1uF_0402" (id 1) (at 154.94 60.96 0)
+      (effects (font (size 0.762 0.762)) (justify left))
+    )
+    (property "Footprint" "Janelia:SM0402" (id 2) (at 153.3652 64.77 0)
+      (effects (font (size 0.762 0.762)) hide)
+    )
+    (property "Datasheet" "" (id 3) (at 152.4 60.96 0)
+      (effects (font (size 1.524 1.524)) hide)
+    )
+    (property "Vendor" "Digi-Key" (id 4) (at 154.94 55.88 0)
+      (effects (font (size 1.524 1.524)) hide)
+    )
+    (property "Vendor Part Number" "311-1375-1-ND" (id 5) (at 157.48 53.34 0)
+      (effects (font (size 1.524 1.524)) hide)
+    )
+    (property "Description" "CAP CER 0.1UF 25V Y5V" (id 6) (at 160.02 50.8 0)
+      (effects (font (size 1.524 1.524)) hide)
+    )
+    (property "Package" "0402" (id 7) (at 152.4 60.96 0)
+      (effects (font (size 1.27 1.27)) hide)
+    )
+    (property "Manufacturer" "Yageo" (id 8) (at 152.4 60.96 0)
+      (effects (font (size 1.27 1.27)) hide)
+    )
+    (property "Manufacturer Part Number" "CC0402ZRY5V8BB104" (id 9) (at 152.4 60.96 0)
+      (effects (font (size 1.27 1.27)) hide)
+    )
+    (pin "1")
+    (pin "2")
+  )
   (symbol (lib_id "Janelia:AS5047P") (at 129.54 96.52 0) (unit 1)
     (in_bom yes) (on_board yes)
-    (property "Reference" "U2" (id 0) (at 137.16 81.28 0)
+    (property "Reference" "U3" (id 0) (at 137.16 81.28 0)
       (effects (font (size 1.524 1.524)) (justify left))
     )
@@
     (pin "9")
   )
-  (symbol (lib_id "Janelia:0.1uF_0402") (at 152.4 60.96 0) (unit 1)
-    (in_bom yes) (on_board yes) (fields_autoplaced)
-    (property "Reference" "C8" (id 0) (at 156.21 60.325 0)
-      (effects (font (size 1.016 1.016)) (justify left))
-    )
-    (property "Value" "0.1uF" (id 1) (at 156.21 62.865 0)
-      (effects (font (size 0.762 0.762)) (justify left))
-    )
-    (property "Footprint" "Janelia:SM0402" (id 2) (at 153.3652 64.77 0)
-      (effects (font (size 0.762 0.762)) hide)
-    )
-    (property "Datasheet" "" (id 3) (at 152.4 60.96 0)
-      (effects (font (size 1.524 1.524)) hide)
-    )
-    (property "Vendor" "Digi-Key" (id 4) (at 154.94 55.88 0)
-      (effects (font (size 1.524 1.524)) hide)
-    )
-    (property "Vendor Part Number" "311-1375-1-ND" (id 5) (at 157.48 53.34 0)
-      (effects (font (size 1.524 1.524)) hide)
-    )
-    (property "Description" "CAP CER 0.1UF 25V Y5V" (id 6) (at 160.02 50.8 0)
-      (effects (font (size 1.524 1.524)) hide)
-    )
-    (property "Package" "0402" (id 7) (at 152.4 60.96 0)
-      (effects (font (size 1.27 1.27)) hide)
-    )
-    (property "Manufacturer" "Yageo" (id 8) (at 152.4 60.96 0)
-      (effects (font (size 1.27 1.27)) hide)
-    )
-    (property "Manufacturer Part Number" "CC0402ZRY5V8BB104" (id 9) (at 152.4 60.96 0)
-      (effects (font (size 1.27 1.27)) hide)
-    )
-    (pin "1")
-    (pin "2")
-  )
 )

Commit message: Add boost for both led and servo
Parts:
- renumbered C11 to C8, U3 to U2
Changed lines of the file:
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@@
   (symbol (lib_id "Janelia:C_0.1uF_0402") (at 152.4 60.96 0) (unit 1)
     (in_bom yes) (on_board yes)
-    (property "Reference" "C11" (id 0) (at 154.94 58.42 0)
+    (property "Reference" "C8" (id 0) (at 154.94 58.42 0)
       (effects (font (size 1.016 1.016)) (justify left))
     )
@@
   (symbol (lib_id "Janelia:AS5047P") (at 129.54 96.52 0) (unit 1)
     (in_bom yes) (on_board yes)
-    (property "Reference" "U3" (id 0) (at 137.16 81.28 0)
+    (property "Reference" "U2" (id 0) (at 137.16 81.28 0)
       (effects (font (size 1.524 1.524)) (justify left))
     )

Commit message: Completed v1.1 layout
Parts:
- C8: value C_0.1uF_0402 -> 0.1uF
Changed lines of the file:
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@@
   (title_block
     (title "biym-board-encoder")
-    (date "2022-11-17")
-    (rev "1.0")
+    (date "2022-11-20")
+    (rev "1.1")
     (company "Peter Polidoro")
   )
@@
       (effects (font (size 1.016 1.016)) (justify left))
     )
-    (property "Value" "C_0.1uF_0402" (id 1) (at 154.94 60.96 0)
+    (property "Value" "0.1uF" (id 1) (at 154.94 60.96 0)
       (effects (font (size 0.762 0.762)) (justify left))
     )

Commit message: Adjust after circuithub import test
Parts:
- U2: Manufacturer ams OSRAM -> Osram
Changed lines of the file:
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@@
       (effects (font (size 1.524 1.524)) hide)
     )
-    (property "Manufacturer" "ams OSRAM" (id 7) (at 129.54 52.07 0)
+    (property "Manufacturer" "Osram" (id 7) (at 129.54 52.07 0)
       (effects (font (size 1.27 1.27)) hide)
     )
