File: biym-board/biym-board.kicad_pcb (KiCad board)
At the start: 2 copper layers, 50.8 x 34 mm, 44 parts, among them J1 HEADER_01X02_JST_ZH_SMD_VERTI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, J2 HEADER_01X03_JST_ZH_SMD_VERTI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, J3 HEADER_01X04_JST_ZH_SMD_VERTI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, J4 HEADER_01X03_JST_ZH_SMD_VERTI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, J5 HEADER_01X03_JST_ZH_SMD_VERTI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, J6 HEADER_01X03_JST_ZH_SMD_VERTI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, P1 POGO_01X04_0.1IN_1_SMD, P2 POGO_01X04_0.1IN_1_SMD, P3 POGO_01X04_0.1IN_1_SMD, P4 POGO_01X04_0.1IN_1_SMD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

Commit message: Update version number
Other:
- board text added: "biym-board v1.3 11/22 peter@polidoro.io https://github.com/biym/biym-board"
- board text removed: "biym-board v1.2 11/22 peter@polidoro.io https://github.com/biym/biym-board"
Changed lines of the file:
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@@
   (title_block
     (title "biym-board")
-    (date "2022-11-20")
-    (rev "1.2")
+    (date "2022-11-29")
+    (rev "1.3")
     (company "Peter Polidoro")
   )
@@
     (effects (font (size 0.5 0.5) (thickness 0.125)) (justify mirror))
   )
-  (gr_text "biym-board\nv1.2 11/22\npeter@polidoro.io\nhttps://github.com/biym/biym-board" (at 140 94.5) (layer "B.SilkS")
+  (gr_text "biym-board\nv1.3 11/22\npeter@polidoro.io\nhttps://github.com/biym/biym-board" (at 140 94.5) (layer "B.SilkS")
     (effects (font (size 0.55 0.5) (thickness 0.1)) (justify mirror))
   )
@@
     (effects (font (size 0.5 0.5) (thickness 0.125)))
   )
-  (gr_text "biym-board\nv1.2 11/22\npeter@polidoro.io\nhttps://github.com/biym/biym-board" (at 123.5 86.75) (layer "F.SilkS")
+  (gr_text "biym-board\nv1.3 11/22\npeter@polidoro.io\nhttps://github.com/biym/biym-board" (at 123.5 86.75) (layer "F.SilkS")
     (effects (font (size 0.55 0.5) (thickness 0.1)))
   )
