File: biym-board/boost.kicad_sch (KiCad schematic)
At the start: 6 parts, among them U4 BOOST_5V_RP402N501F

Commit message: Completed v1.1 layout
Parts:
- C11, C12, C13: value C_10uF_0603 -> 10uF
- R2: value R_5.1k_0402 -> 5.1k
Other:
- company: (none) -> Peter Polidoro
Changed lines of the file:
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@@
   (title_block
     (title "biym-board-power-boost")
-    (rev "1.0")
+    (date "2022-11-20")
+    (rev "1.1")
+    (company "Peter Polidoro")
   )
   (wire (pts (xy 118.11 102.87) (xy 120.65 102.87))
@@
       (effects (font (size 1.016 1.016)) (justify left))
     )
-    (property "Value" "R_5.1k_0402" (id 1) (at 101.6 116.84 0)
+    (property "Value" "5.1k" (id 1) (at 101.6 116.84 0)
       (effects (font (size 0.762 0.762)) (justify left))
     )
@@
       (effects (font (size 1.016 1.016)) (justify left))
     )
-    (property "Value" "C_10uF_0603" (id 1) (at 102.87 85.09 0)
+    (property "Value" "10uF" (id 1) (at 102.87 85.09 0)
       (effects (font (size 0.762 0.762)) (justify left))
     )
@@
       (effects (font (size 1.016 1.016)) (justify left))
     )
-    (property "Value" "C_10uF_0603" (id 1) (at 157.48 87.63 0)
+    (property "Value" "10uF" (id 1) (at 157.48 87.63 0)
       (effects (font (size 0.762 0.762)) (justify left))
     )
@@
       (effects (font (size 1.016 1.016)) (justify left))
     )
-    (property "Value" "C_10uF_0603" (id 1) (at 173.99 87.63 0)
-      (effects (font (size 0.762 0.762)) (justify left))
-    )
+    (property "Value" "10uF" (id 1) (at 173.99 87.63 0)
+      (effects (font (size 0.762 0.762)) (justify left))
+    )

Commit message: Update to kicad 7
Other:
- title: biym-board-power-boost -> biym-board
