File: biym-board/featherwing-nrf52-pogo.kicad_sch (KiCad schematic)
At the start: 3 parts, among them P1 POGO_01X16_0.1IN_1_SMD, P2 POGO_01X12_0.1IN_1_SMD

Commit message: Adjust after circuithub import test
Parts:
- FW1: now left out of the parts list
Changed lines of the file:
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@@
   )
   (symbol (lib_id "Janelia:FEATHERWING_nRF52") (at 143.51 99.06 0) (unit 1)
-    (in_bom yes) (on_board yes)
+    (in_bom no) (on_board yes)
     (property "Reference" "FW1" (id 0) (at 143.51 73.66 0))
     (property "Value" "FEATHERWING_nRF52" (id 1) (at 143.51 124.46 0))

Commit message: Finished v1.2
Parts:
- removed P1: POGO_01X16_0.1IN_1_SMD, Janelia:POGO_01x16_0.1in_SMD, symbol Janelia:POGO_01X16_0.1IN_1_SMD
- removed P2: POGO_01X12_0.1IN_1_SMD, Janelia:POGO_01x12_0.1in_SMD, symbol Janelia:POGO_01X12_0.1IN_1_SMD
- added P1, P2, P3, P4, P5, P6, P7: POGO_01X04_0.1IN_1_SMD, Janelia:POGO_01x04_0.1in_SMD, symbol Janelia:POGO_01X04_0.1IN_1_SMD
Connections:
- net ENABLE_VREG: now also P7.3 (P3)
- net GND: now also P1.4 (P4)
- net GPIO/0/TX-HS: now also P4.3 (P3)
- net GPIO/10-HS: now also P6.2 (P2)
- net GPIO/11-HS: now also P6.3 (P3)
- net GPIO/12-HS: now also P6.4 (P4)
- net GPIO/13-HS: now also P7.1 (P1)
- net GPIO/14/A0-HS: now also P2.1 (P1)
- net GPIO/15/A1-HS: now also P2.2 (P2)
- net GPIO/16/A2-LS: now also P2.3 (P3)
- net GPIO/17/A3-LS: now also P2.4 (P4)
- net GPIO/18/A4-LS: now also P3.1 (P1)
- net GPIO/19/A5-LS: now also P3.2 (P2)
- net GPIO/1/RX-HS: now also P4.2 (P2)
- net GPIO/21/AREF/A7-LS: now also P1.3 (P3)
- net GPIO/22/SDA-HS: now also P5.1 (P1)
- net GPIO/23/SCL-HS: now also P5.2 (P2)
- net GPIO/24/MISO-HS: now also P4.1 (P1)
- net GPIO/25/MOSI-HS: now also P3.4 (P4)
- net GPIO/26/SCK-HS: now also P3.3 (P3)
- net GPIO/2/NFC2-LS: now also P4.4 (P4)
- net GPIO/5-HS: now also P5.3 (P3)
- net GPIO/6-HS: now also P5.4 (P4)
- net GPIO/9-HS: now also P6.1 (P1)
- net V3.3: now also P1.2 (P2)
- net VBATTERY: now also P7.4 (P4)
- net VUSB: now also P7.2 (P2)
- net ~{RESET}: now also P1.1 (P1)

Commit message: Update to kicad 7
Other:
- title: biym-board-featherwing -> biym-board
