File: biym-board/led.kicad_sch (KiCad schematic)
At the start: 1 part, among them J3 HEADER_01X04_JST_ZH_SMD_VERTI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

Commit message: Update to kicad 7
Other:
- title: biym-board-led -> biym-board
Changed lines of the file:
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@@
-(kicad_sch (version 20211123) (generator eeschema)
+(kicad_sch (version 20230121) (generator eeschema)
   (paper "A4")
   (title_block
-    (title "biym-board-led")
-    (date "2022-11-29")
+    (title "biym-board")
+    (date "2024-05-16")
     (rev "1.3")
     (company "Peter Polidoro")
   )
   (wire (pts (xy 139.7 96.52) (xy 142.24 96.52))
-    (stroke (width 0) (type default) (color 0 0 0 0))
+    (stroke (width 0) (type default))
   )
   (wire (pts (xy 139.7 93.98) (xy 142.24 93.98))
-    (stroke (width 0) (type default) (color 0 0 0 0))
+    (stroke (width 0) (type default))
   )
   (wire (pts (xy 139.7 99.06) (xy 142.24 99.06))
-    (stroke (width 0) (type default) (color 0 0 0 0))
+    (stroke (width 0) (type default))
   )
   (wire (pts (xy 139.7 101.6) (xy 142.24 101.6))
-    (stroke (width 0) (type default) (color 0 0 0 0))
+    (stroke (width 0) (type default))
   )
-  (hierarchical_label "VLED" (shape passive) (at 139.7 93.98 180)
+  (hierarchical_label "VLED" (shape passive) (at 139.7 93.98 180) (fields_autoplaced)
     (effects (font (size 1.27 1.27)) (justify right))
   )
-  (hierarchical_label "SDI" (shape input) (at 139.7 99.06 180)
+  (hierarchical_label "SDI" (shape input) (at 139.7 99.06 180) (fields_autoplaced)
     (effects (font (size 1.27 1.27)) (justify right))
   )
-  (hierarchical_label "GND" (shape passive) (at 139.7 101.6 180)
+  (hierarchical_label "GND" (shape passive) (at 139.7 101.6 180) (fields_autoplaced)
     (effects (font (size 1.27 1.27)) (justify right))
   )
-  (hierarchical_label "CKI" (shape input) (at 139.7 96.52 180)
+  (hierarchical_label "CKI" (shape input) (at 139.7 96.52 180) (fields_autoplaced)
     (effects (font (size 1.27 1.27)) (justify right))
   )
   (symbol (lib_id "Janelia:HEADER_01X04_JST_ZH_SMD_VERTICAL") (at 147.32 97.79 180) (unit 1)
-    (in_bom yes) (on_board yes)
-    (property "Reference" "J3" (id 0) (at 147.32 91.44 0))
-    (property "Value" "HEADER_01X04_JST_ZH_SMD_VERTICAL" (id 1) (at 147.32 104.14 0))
-    (property "Footprint" "Janelia:JST_ZH_B4B_ZR_SM4_TF_1x04-1MP_P1.50mm_Vertical" (id 2) (at 147.32 110.49 0)
+    (in_bom yes) (on_board yes) (dnp no)
+    (property "Reference" "J3" (at 147.32 91.44 0)
+      (effects (font (size 1.27 1.27)))
+    )
+    (property "Value" "HEADER_01X04_JST_ZH_SMD_VERTICAL" (at 147.32 104.14 0)
+      (effects (font (size 1.27 1.27)))
+    )
+    (property "Footprint" "Janelia:JST_ZH_B4B_ZR_SM4_TF_1x04-1MP_P1.50mm_Vertical" (at 147.32 110.49 0)
       (effects (font (size 1.27 1.27)) hide)
     )
-    (property "Datasheet" "" (id 3) (at 147.32 99.06 0)
+    (property "Datasheet" "" (at 147.32 99.06 0)
       (effects (font (size 1.27 1.27)) hide)
     )
-    (property "Description" "CONN HEADER SMD 4POS 1.5MM" (id 4) (at 147.32 107.95 0)
+    (property "Description" "CONN HEADER SMD 4POS 1.5MM" (at 147.32 107.95 0)
       (effects (font (size 1.27 1.27)) hide)
     )
-    (property "Manufacturer" "JST Sales America Inc." (id 5) (at 147.32 115.57 0)
+    (property "Manufacturer" "JST Sales America Inc." (at 147.32 115.57 0)
       (effects (font (size 1.27 1.27)) hide)
     )
-    (property "Manufacturer Part Number" "B4B-ZR-SM4-TF(LF)(SN)" (id 6) (at 147.32 113.03 0)
+    (property "Manufacturer Part Number" "B4B-ZR-SM4-TF(LF)(SN)" (at 147.32 113.03 0)
       (effects (font (size 1.27 1.27)) hide)
     )
-    (property "Vendor" "Digi-Key" (id 7) (at 147.32 118.11 0)
+    (property "Vendor" "Digi-Key" (at 147.32 118.11 0)
       (effects (font (size 1.27 1.27)) hide)
     )
-    (property "Vendor Part Number" "455-1683-1-ND" (id 8) (at 147.32 120.65 0)
+    (property "Vendor Part Number" "455-1683-1-ND" (at 147.32 120.65 0)
       (effects (font (size 1.27 1.27)) hide)
     )
@@
     (pin "3")
     (pin "4")
+    (instances
+      (project "biym-board"
+        (path "/8aa5116f-ac54-4325-a42a-36123c2901d1/ba7902c8-ef45-407b-94b0-d9c747cdabc9"
+          (reference "J3") (unit 1)
+        )
+      )
+    )
   )
 )
