File: biym-board/servo.kicad_sch (KiCad schematic)
At the start: 3 parts

Commit message: Finished v0.1 of schematic
Parts:
- removed C? (x2): 0.1uF, Janelia:SM0402, symbol Janelia:0.1uF_0402
- added C14, C15: C_0.1uF_0402, Janelia:SM0402, symbol Janelia:C_0.1uF_0402
- added J4, J5: HEADER_01X03_JST_ZH_SMD_VERTICAL, Janelia:JST_ZH_B3B_ZR_SM4_TF_1x03-1MP_P1.50mm_Vertical, symbol Janelia:HEADER_01X03_JST_ZH_SMD_VERTICAL
- gave numbers to parts that had none: 1
Connections:
- net GND: now also C14.2, C15.2, J4.3 (Pin_3), J5.3 (Pin_3)
- net TRANSLATED_SIGNAL_0: now also J4.1 (Pin_1)
- net TRANSLATED_SIGNAL_1: now also J5.1 (Pin_1)
- net VDIGITAL: now also C14.1
- net VSERVO: now also C15.1, J4.2 (Pin_2), J5.2 (Pin_2)
Other:
- company: (none) -> Peter Polidoro
- title: (none) -> biym-board-servo
Changed lines of the file:
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@@
 (kicad_sch (version 20211123) (generator eeschema)
   (paper "A4")
-  (wire (pts (xy 147.32 71.12) (xy 147.32 73.66))
+  (title_block
+    (title "biym-board-servo")
+    (date "2022-11-17")
+    (rev "0.1")
+    (company "Peter Polidoro")
+  )
+  (wire (pts (xy 195.58 99.06) (xy 198.12 99.06))
+    (stroke (width 0) (type default) (color 0 0 0 0))
+  )
+  (wire (pts (xy 149.86 71.12) (xy 149.86 73.66))
+    (stroke (width 0) (type default) (color 0 0 0 0))
+  )
+  (wire (pts (xy 195.58 114.3) (xy 198.12 114.3))
     (stroke (width 0) (type default) (color 0 0 0 0))
   )
@@
     (stroke (width 0) (type default) (color 0 0 0 0))
   )
-  (wire (pts (xy 147.32 83.82) (xy 147.32 86.36))
+  (wire (pts (xy 149.86 83.82) (xy 149.86 86.36))
     (stroke (width 0) (type default) (color 0 0 0 0))
   )
@@
     (stroke (width 0) (type default) (color 0 0 0 0))
   )
+  (wire (pts (xy 195.58 96.52) (xy 198.12 96.52))
+    (stroke (width 0) (type default) (color 0 0 0 0))
+  )
   (wire (pts (xy 97.79 106.68) (xy 100.33 106.68))
     (stroke (width 0) (type default) (color 0 0 0 0))
@@
     (stroke (width 0) (type default) (color 0 0 0 0))
   )
+  (wire (pts (xy 195.58 116.84) (xy 198.12 116.84))
+    (stroke (width 0) (type default) (color 0 0 0 0))
+  )
+  (wire (pts (xy 195.58 93.98) (xy 198.12 93.98))
+    (stroke (width 0) (type default) (color 0 0 0 0))
+  )
+  (wire (pts (xy 195.58 111.76) (xy 198.12 111.76))
+    (stroke (width 0) (type default) (color 0 0 0 0))
+  )
   (text "DIR: A -> B" (at 88.9 111.76 180)
     (effects (font (size 1.27 1.27)) (justify right bottom))
@@
     (effects (font (size 1.27 1.27)) (justify right bottom))
   )
+  (label "VSERVO" (at 195.58 96.52 180)
+    (effects (font (size 1.27 1.27)) (justify right bottom))
+  )
   (label "VDIGITAL" (at 134.62 71.12 0)
     (effects (font (size 1.27 1.27)) (justify left bottom))
@@
     (effects (font (size 1.27 1.27)) (justify right bottom))
   )
-  (label "VSERVO" (at 147.32 71.12 0)
-    (effects (font (size 1.27 1.27)) (justify left bottom))
+  (label "VSERVO" (at 149.86 71.12 0)
+    (effects (font (size 1.27 1.27)) (justify left bottom))
+  )
+  (label "VSERVO" (at 195.58 114.3 180)
+    (effects (font (size 1.27 1.27)) (justify right bottom))
   )
   (label "TRANSLATED_SIGNAL_1" (at 123.19 106.68 0)
     (effects (font (size 1.27 1.27)) (justify left bottom))
   )
+  (label "GND" (at 195.58 93.98 180)
+    (effects (font (size 1.27 1.27)) (justify right bottom))
+  )
   (label "TRANSLATED_SIGNAL_0" (at 123.19 101.6 0)
     (effects (font (size 1.27 1.27)) (justify left bottom))
   )
+  (label "TRANSLATED_SIGNAL_1" (at 195.58 116.84 180)
+    (effects (font (size 1.27 1.27)) (justify right bottom))
+  )
   (label "VDIGITAL" (at 80.01 82.55 0)
     (effects (font (size 1.27 1.27)) (justify left bottom))
@@
     (effects (font (size 1.27 1.27)) (justify left bottom))
   )
+  (label "GND" (at 195.58 111.76 180)
+    (effects (font (size 1.27 1.27)) (justify right bottom))
+  )
+  (label "TRANSLATED_SIGNAL_0" (at 195.58 99.06 180)
+    (effects (font (size 1.27 1.27)) (justify right bottom))
+  )
   (label "GND" (at 110.49 119.38 0)
     (effects (font (size 1.27 1.27)) (justify left bottom))
   )
-  (label "GND" (at 147.32 86.36 0)
+  (label "GND" (at 149.86 86.36 0)
     (effects (font (size 1.27 1.27)) (justify left bottom))
   )
@@
     (effects (font (size 1.27 1.27)) (justify right))
   )
-  (symbol (lib_id "Janelia:0.1uF_0402") (at 134.62 78.74 0) (unit 1)
-    (in_bom yes) (on_board yes) (fields_autoplaced)
-    (property "Reference" "C?" (id 0) (at 138.43 78.105 0)
+  (symbol (lib_id "Janelia:C_0.1uF_0402") (at 134.62 78.74 0) (unit 1)
+    (in_bom yes) (on_board yes)
+    (property "Reference" "C14" (id 0) (at 137.16 76.2 0)
       (effects (font (size 1.016 1.016)) (justify left))
     )
-    (property "Value" "0.1uF" (id 1) (at 138.43 80.645 0)
+    (property "Value" "C_0.1uF_0402" (id 1) (at 137.16 78.74 0)
       (effects (font (size 0.762 0.762)) (justify left))
     )
@@
     (pin "2")
   )
-  (symbol (lib_id "Janelia:0.1uF_0402") (at 147.32 78.74 0) (unit 1)
-    (in_bom yes) (on_board yes) (fields_autoplaced)
-    (property "Reference" "C?" (id 0) (at 151.13 78.105 0)
+  (symbol (lib_id "Janelia:HEADER_01X03_JST_ZH_SMD_VERTICAL") (at 203.2 114.3 180) (unit 1)
+    (in_bom yes) (on_board yes)
+    (property "Reference" "J5" (id 0) (at 203.2 109.22 0))
+    (property "Value" "HEADER_01X03_JST_ZH_SMD_VERTICAL" (id 1) (at 203.2 119.38 0))
+    (property "Footprint" "Janelia:JST_ZH_B3B_ZR_SM4_TF_1x03-1MP_P1.50mm_Vertical" (id 2) (at 203.2 127 0)
+      (effects (font (size 1.27 1.27)) hide)
+    )
+    (property "Datasheet" "" (id 3) (at 203.2 114.3 0)
+      (effects (font (size 1.27 1.27)) hide)
+    )
+    (property "Description" "CONN HEADER SMD 3POS 1.5MM" (id 4) (at 203.2 124.46 0)
+      (effects (font (size 1.27 1.27)) hide)
+    )
+    (property "Manufacturer" "JST Sales America Inc." (id 5) (at 203.2 132.08 0)
+      (effects (font (size 1.27 1.27)) hide)
+    )
+    (property "Manufacturer Part Number" "B3B-ZR-SM4-TF(LF)(SN)" (id 6) (at 203.2 129.54 0)
+      (effects (font (size 1.27 1.27)) hide)
+    )
+    (property "Vendor" "Digi-Key" (id 7) (at 203.2 134.62 0)
+      (effects (font (size 1.27 1.27)) hide)
+    )
+    (property "Vendor Part Number" "B3B-ZR-SM4-TF(LF)(SN)" (id 8) (at 203.2 137.16 0)
+      (effects (font (size 1.27 1.27)) hide)
+    )
+    (pin "1")
+    (pin "2")
+    (pin "3")
+  )
+  (symbol (lib_id "Janelia:C_0.1uF_0402") (at 149.86 78.74 0) (unit 1)
+    (in_bom yes) (on_board yes)
+    (property "Reference" "C15" (id 0) (at 152.4 76.2 0)
       (effects (font (size 1.016 1.016)) (justify left))
     )
-    (property "Value" "0.1uF" (id 1) (at 151.13 80.645 0)
+    (property "Value" "C_0.1uF_0402" (id 1) (at 152.4 78.74 0)
       (effects (font (size 0.762 0.762)) (justify left))
     )
-    (property "Footprint" "Janelia:SM0402" (id 2) (at 148.2852 82.55 0)
+    (property "Footprint" "Janelia:SM0402" (id 2) (at 150.8252 82.55 0)
       (effects (font (size 0.762 0.762)) hide)
     )
-    (property "Datasheet" "" (id 3) (at 147.32 78.74 0)
-      (effects (font (size 1.524 1.524)) hide)
-    )
-    (property "Vendor" "Digi-Key" (id 4) (at 149.86 73.66 0)
-      (effects (font (size 1.524 1.524)) hide)
-    )
-    (property "Vendor Part Number" "311-1375-1-ND" (id 5) (at 152.4 71.12 0)
-      (effects (font (size 1.524 1.524)) hide)
-    )
-    (property "Description" "CAP CER 0.1UF 25V Y5V" (id 6) (at 154.94 68.58 0)
-      (effects (font (size 1.524 1.524)) hide)
-    )
-    (property "Package" "0402" (id 7) (at 147.32 78.74 0)
-      (effects (font (size 1.27 1.27)) hide)
-    )
-    (property "Manufacturer" "Yageo" (id 8) (at 147.32 78.74 0)
-      (effects (font (size 1.27 1.27)) hide)
-    )
-    (property "Manufacturer Part Number" "CC0402ZRY5V8BB104" (id 9) (at 147.32 78.74 0)
+    (property "Datasheet" "" (id 3) (at 149.86 78.74 0)
+      (effects (font (size 1.524 1.524)) hide)
+    )
+    (property "Vendor" "Digi-Key" (id 4) (at 152.4 73.66 0)
+      (effects (font (size 1.524 1.524)) hide)
+    )
+    (property "Vendor Part Number" "311-1375-1-ND" (id 5) (at 154.94 71.12 0)
+      (effects (font (size 1.524 1.524)) hide)
+    )
+    (property "Description" "CAP CER 0.1UF 25V Y5V" (id 6) (at 157.48 68.58 0)
+      (effects (font (size 1.524 1.524)) hide)
+    )
+    (property "Package" "0402" (id 7) (at 149.86 78.74 0)
+      (effects (font (size 1.27 1.27)) hide)
+    )
+    (property "Manufacturer" "Yageo" (id 8) (at 149.86 78.74 0)
+      (effects (font (size 1.27 1.27)) hide)
+    )
+    (property "Manufacturer Part Number" "CC0402ZRY5V8BB104" (id 9) (at 149.86 78.74 0)
       (effects (font (size 1.27 1.27)) hide)
     )
@@
   (symbol (lib_id "Janelia:LT_SN74LVC2T45DCUT") (at 110.49 104.14 0) (unit 1)
     (in_bom yes) (on_board yes)
-    (property "Reference" "U?" (id 0) (at 116.84 92.71 0)
+    (property "Reference" "U4" (id 0) (at 116.84 92.71 0)
       (effects (font (size 1.27 1.27)) (justify left))
     )
@@
     (pin "8")
   )
+  (symbol (lib_id "Janelia:HEADER_01X03_JST_ZH_SMD_VERTICAL") (at 203.2 96.52 180) (unit 1)
+    (in_bom yes) (on_board yes)
+    (property "Reference" "J4" (id 0) (at 203.2 91.44 0))
+    (property "Value" "HEADER_01X03_JST_ZH_SMD_VERTICAL" (id 1) (at 203.2 101.6 0))
+    (property "Footprint" "Janelia:JST_ZH_B3B_ZR_SM4_TF_1x03-1MP_P1.50mm_Vertical" (id 2) (at 203.2 109.22 0)
+      (effects (font (size 1.27 1.27)) hide)
+    )
+    (property "Datasheet" "" (id 3) (at 203.2 96.52 0)
+      (effects (font (size 1.27 1.27)) hide)
+    )
+    (property "Description" "CONN HEADER SMD 3POS 1.5MM" (id 4) (at 203.2 106.68 0)
+      (effects (font (size 1.27 1.27)) hide)
+    )
+    (property "Manufacturer" "JST Sales America Inc." (id 5) (at 203.2 114.3 0)
+      (effects (font (size 1.27 1.27)) hide)
+    )
+    (property "Manufacturer Part Number" "B3B-ZR-SM4-TF(LF)(SN)" (id 6) (at 203.2 111.76 0)
+      (effects (font (size 1.27 1.27)) hide)
+    )
+    (property "Vendor" "Digi-Key" (id 7) (at 203.2 116.84 0)
+      (effects (font (size 1.27 1.27)) hide)
+    )
+    (property "Vendor Part Number" "B3B-ZR-SM4-TF(LF)(SN)" (id 8) (at 203.2 119.38 0)
+      (effects (font (size 1.27 1.27)) hide)
+    )
+    (pin "1")
+    (pin "2")
+    (pin "3")
+  )
 )

Commit message: Add boost for both led and servo
Parts:
- renumbered C15 to C10, C14 to C9, U4 to U3
Changed lines of the file:
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@@
   (symbol (lib_id "Janelia:C_0.1uF_0402") (at 134.62 78.74 0) (unit 1)
     (in_bom yes) (on_board yes)
-    (property "Reference" "C14" (id 0) (at 137.16 76.2 0)
+    (property "Reference" "C9" (id 0) (at 137.16 76.2 0)
       (effects (font (size 1.016 1.016)) (justify left))
     )
@@
   (symbol (lib_id "Janelia:C_0.1uF_0402") (at 149.86 78.74 0) (unit 1)
     (in_bom yes) (on_board yes)
-    (property "Reference" "C15" (id 0) (at 152.4 76.2 0)
+    (property "Reference" "C10" (id 0) (at 152.4 76.2 0)
       (effects (font (size 1.016 1.016)) (justify left))
     )
@@
   (symbol (lib_id "Janelia:LT_SN74LVC2T45DCUT") (at 110.49 104.14 0) (unit 1)
     (in_bom yes) (on_board yes)
-    (property "Reference" "U4" (id 0) (at 116.84 92.71 0)
+    (property "Reference" "U3" (id 0) (at 116.84 92.71 0)
       (effects (font (size 1.27 1.27)) (justify left))
     )

Commit message: Completed v1.1 layout
Parts:
- C10, C9: value C_0.1uF_0402 -> 0.1uF
Changed lines of the file:
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@@
   (title_block
     (title "biym-board-servo")
-    (date "2022-11-17")
-    (rev "1.0")
+    (date "2022-11-20")
+    (rev "1.1")
     (company "Peter Polidoro")
   )
@@
       (effects (font (size 1.016 1.016)) (justify left))
     )
-    (property "Value" "C_0.1uF_0402" (id 1) (at 137.16 78.74 0)
+    (property "Value" "0.1uF" (id 1) (at 137.16 78.74 0)
       (effects (font (size 0.762 0.762)) (justify left))
     )
@@
       (effects (font (size 1.016 1.016)) (justify left))
     )
-    (property "Value" "C_0.1uF_0402" (id 1) (at 152.4 78.74 0)
+    (property "Value" "0.1uF" (id 1) (at 152.4 78.74 0)
       (effects (font (size 0.762 0.762)) (justify left))
     )

Commit message: Update to kicad 7
Other:
- title: biym-board-servo -> biym-board
